File: hw/kicad/cell.kicad_sch (KiCad schematic)
At the start: 14 parts, among them Q1012 DMMT5551, Q301 THAT300, U1011 SN74LVC1G74

Commit message: Select analog thermal packages and document carrier layout
Parts:
- U1011: footprint Package_SO:VSSOP-8_2.3x2mm_P0.5mm -> bfdac:TI_DQE_X2SON-8_1.4x1.0mm_P0.35mm; MPN SN74LVC1G74DCUR -> SN74LVC1G74DQER
