File: hw/kicad/cell_r.kicad_sch (KiCad schematic)
At the start: 14 parts, among them Q2012 DMMT5551, Q401 THAT300, U2011 SN74LVC1G74

Commit message: Select analog thermal packages and document carrier layout
Parts:
- U2011: footprint Package_SO:VSSOP-8_2.3x2mm_P0.5mm -> bfdac:TI_DQE_X2SON-8_1.4x1.0mm_P0.35mm; MPN SN74LVC1G74DCUR -> SN74LVC1G74DQER
