File: hw/kicad/iv_r.kicad_sch (KiCad schematic)
At the start: 52 parts, among them U61 OPA1612, U62 OPA1612, U63 BUF634A, U64 BUF634A, U785 LT3045

Commit message: Select analog thermal packages and document carrier layout
Parts:
- U61, U62: footprint Package_SO:SOIC-8_3.9x4.9mm_P1.27mm -> bfdac:TI_OPA1612_DRG_WSON-8_3x3mm_P0.5mm_EP1.2x2.0mm; MPN OPA1612AIDR -> OPA1612AIDRGR
- U63, U64: footprint Package_SO:SOIC-8_3.9x4.9mm_P1.27mm -> bfdac:TI_BUF634A_DDA_HSOIC-8_P1.27mm_EP2.95x4.9mm; MPN BUF634AIDR -> BUF634AIDDAR
