File: hw/kicad/refs.kicad_sch (KiCad schematic)
At the start: 147 parts, among them Q901 BCP56-16, Q902 2SA1036K, Q903 BC817-40, Q904 BC807-40, Q905 BC847B, U901 REF7050, U902 OPA1656, U903 OPA1612, U904 OPA1612, U905 OPA1612, U906 LT3045, U907 OPA1656, U908 LT3045, U909 LT3045, U910 LT3094, U911 LT3094

Commit message: Select analog thermal packages and document carrier layout
Parts:
- U903, U904, U905: footprint Package_SO:SOIC-8_3.9x4.9mm_P1.27mm -> bfdac:TI_OPA1612_DRG_WSON-8_3x3mm_P0.5mm_EP1.2x2.0mm; MPN OPA1612AIDR -> OPA1612AIDRGR
