File: hw/kicad/refs_r.kicad_sch (KiCad schematic)
At the start: 137 parts, among them Q701 BCP56-16, Q702 2SA1036K, Q703 BC817-40, Q704 BC807-40, Q705 BC847B, U702 OPA1656, U703 OPA1612, U704 OPA1612, U705 OPA1612, U706 LT3045, U707 OPA1656, U708 LT3045, U709 LT3045, U710 LT3094, U711 LT3094

Commit message: Select analog thermal packages and document carrier layout
Parts:
- U703, U704, U705: footprint Package_SO:SOIC-8_3.9x4.9mm_P1.27mm -> bfdac:TI_OPA1612_DRG_WSON-8_3x3mm_P0.5mm_EP1.2x2.0mm; MPN OPA1612AIDR -> OPA1612AIDRGR
